File: Super_Dolly_Board.sch (EAGLE design)
At the start: 84 parts, among them J1 10118193-0001LF, J3 SJ1-2503A, J4 RJHS-538X, J5 SJ1-2503A, P1 TC33X-2, SW1 SKQUDBE010, U1 ATMEGA32U4-XUAU, U2 MMDT3904, U3 TB6559FG, U4 LM2937IMP-5.0/NOPB, U5 TB6559FG, U6 SN75176BDR, U7 TB6559FG, U8 TPD2E007DCK, U9 LM2937IMP-5.0/NOPB, X1 3.2X2.5MMCRYSTAL

Commit message: checking in changed to the SDB and adding 2 libraries
Parts:
- added C22: 1uF, parkers_parts:CAP_NONPOL0402
- added C23: .1uF, parkers_parts:CAP_NONPOL0402
- added IC1: AT90USB646-AU, at90usb:AT90USB647-AU
- added R22, R24: 0, parkers_parts:RESISTOR0402
- added R25: 36K, parkers_parts:RESISTOR0402
- added R26: 20K, parkers_parts:RESISTOR0402
- added R27: 10K, parkers_parts:RESISTOR0402
- added S1, S2: SKHHAJA010, SparkFun-Electromechanical:SWITCH-MOMENTARY-2PTH
- C14, C6: value 1uF -> .1uF
- U1: value ATMEGA32U4-XUAU -> AT90USB646-MU; device SmartPrj:ATMEGA32U4-XUAU -> at90usb:AT90USB647-MU
- U4, U9: value LM2937IMP-5.0/NOPB -> TS2937CW50
Connections:
- removed net D0/RX: U1.(RXD1/AIN1/INT2)PD2, U6.R
- removed net D1/TX: U1.(TXD1/INT3)PD3, U6.D
- removed net HWB: U1.(#HWB)PE2
- removed net MISO/M2_P: J2.1, U1.(PD0/MISO/PCINT3)PB3, U3.PWM
- removed net MOSI/M1_P: J2.4, U1.(PDI/MOSI/PCINT2)PB2, U7.PWM
- removed net RESET: J2.5, R11.2, U1.RESET
- removed net RXLED/IO_2: CG3.2, J3.R, U1.(SS/PCINT0)PB0
- removed net SCK/M0_P: J2.3, U1.(SCLK/PCINT1)PB1, U5.PWM
- removed net TXLED: U1.(XCK1/#CTS)PD5
- removed net XTAL1: C4.2, U1.XTAL1, X1.3
- removed net XTAL2: C3.2, U1.XTAL2, X1.1
- new net AGND: C23.2, IC1.GND@3, R24.2, U1.GND@3
- new net BATT_V: IC1.PF1(ADC1), R25.1, R26.2, U1.PF1(ADC1)
- new net IO_0: IC1.PB4(PCINT4/OC.2A), U1.PB4(PCINT4/OC.2A)
- new net IO_1: IC1.PB5(PCINT5/OC.1A), U1.PB5(PCINT5/OC.1A)
- new net IO_2: CG3.2, IC1.PB6(PCINT6/OC.1B), J3.R, U1.PB6(PCINT6/OC.1B)
- new net M0_P: IC1.PA0(AD0), U1.PA0(AD0), U5.PWM
- new net M1_P: IC1.PA1(AD1), U1.PA1(AD1), U7.PWM
- new net M2_P: IC1.PA2(AD2), U1.PA2(AD2), U3.PWM
- new net MISO: IC1.PB3(PDO/PCINT3/MISO), J2.1, U1.PB3(PDO/PCINT3/MISO)
- new net MOSI: IC1.PB2(PDI/PCINT2/MOSI), J2.4, U1.PB2(PDI/PCINT2/MOSI)
- new net PC7: IC1.PC7(A15/IC.3/CLK0), U1.PC7(A15/IC.3/CLK0)
- new net PE0: IC1.PE0(/WR), U1.PE0(/WR)
- new net PE1: IC1.PE1(/RD), U1.PE1(/RD)
- new net PE2: IC1.PE2(ALE/HWB), R27.2, S2.1, U1.PE2(ALE/HWB)
- new net PE3: IC1.PE3(IUID), U1.PE3(IUID)
- new net PE4: IC1.PE4(INT4/TOSC1), U1.PE4(INT4/TOSC1)
- new net PE5: IC1.PE5(INT5/TOSC2), U1.PE5(INT5/TOSC2)
- new net PE6: IC1.PE6(INT6/AIN0), U1.PE6(INT6/AIN0)
- new net PE7: IC1.PE7(INT7/AIN1/UVCON), U1.PE7(INT7/AIN1/UVCON)
- new net PF2: IC1.PF2(ADC2), U1.PF2(ADC2)
- new net PF3: IC1.PF3(ADC3), U1.PF3(ADC3)
- new net PF4: IC1.PF4(ADC4/TCK), U1.PF4(ADC4/TCK)
- new net PF5: IC1.PF5(ADC5/TMS), U1.PF5(ADC5/TMS)
- new net PF6: IC1.PF6(ADC6/TDO), U1.PF6(ADC6/TDO)
- new net PF7: IC1.PF7(ADC7/TDI), U1.PF7(ADC7/TDI)
- new net RST: IC1.RESET, J2.5, R11.2, S1.1, U1.RESET
- new net RX: IC1.PD2(RXD1/INT2), U1.PD2(RXD1/INT2), U6.R
- new net SCK: IC1.PB1(PCINT1/SCK), J2.3, U1.PB1(PCINT1/SCK)
- new net TX: IC1.PD3(TXD1/INT3), U1.PD3(TXD1/INT3), U6.D
- new net UGND: C22.1, CG1.1, CG2.1, CG7.1, IC1.UGND, J1.GND, R22.1, U1.UGND
- new net X1: C4.2, IC1.XTAL1, U1.XTAL1, X1.3
- new net X2: C3.2, IC1.XTAL2, U1.XTAL2, X1.1
- net +5V: now also C5.1, C6.1, IC1.AVCC, IC1.UVCC, IC1.VCC@1, IC1.VCC@2, R27.1, U1.VCC@1, U1.VCC@2; no longer U1.AVCC1, U1.VCC, U1.VCC1
- net AREF: now also C23.1, IC1.AREF; no longer C5.1
- net BTNS: now also IC1.PF0(ADC0), U1.PF0(ADC0); no longer U1.(ADC0)PF0
- net COM1: now also IC1.PD0(OC.0B/SCL/INT0), U1.PD0(OC.0B/SCL/INT0)
- net COM2: now also IC1.PD1(OC.2B/SDA/INT1), U1.PD1(OC.2B/SDA/INT1)
- net COM3: now also IC1.PD7(T0), U1.PD7(T0)
- net DE: now also IC1.PD4(ICP1), U1.PD4(ICP1); no longer U1.(ADC5/TMS)PF5
- net FOC: now also IC1.PD6(T1), U1.PD6(T1); no longer U1.(ADC4/TCK)PF4
- net GND: now also IC1.GND@1, IC1.GND@2, R22.2, R24.1, R26.1, S1.2, S2.2, U1.GND@1, U1.GND@2; no longer CG1.1, CG2.1, CG7.1, J1.GND, U1.GND, U1.GND1, U1.GND2, U1.GND3, U1.PAD, U1.UGND
- net IO_3: now also IC1.PB7(PCINT7/OC.0A/OC.1C), U1.PB7(PCINT7/OC.0A/OC.1C); no longer U1.(SDA/INT1)PD1
- net LCD_BK: now also IC1.PC6(A14/OC.3A), U1.PC6(A14/OC.3A); no longer U1.(ADC6/TDO)PF6
- net LCD_D4: now also IC1.PC0(A8), U1.PC0(A8); no longer U1.(ADC7/TDI)PF7
- net LCD_D5: now also IC1.PC1(A9), U1.PC1(A9); no longer U1.(OC0B/SCL/INT0)PD0
- net LCD_D6: now also IC1.PC2(A10), U1.PC2(A10); no longer U1.(ICP1/ADC8)PD4
- net LCD_D7: now also IC1.PC3(A11/T.3), U1.PC3(A11/T.3); no longer U1.(OC3A/#0C4A)PC6
- net LCD_E: now also IC1.PC4(A12/OC.3C), U1.PC4(A12/OC.3C); no longer U1.(T0/OC4D/ADC10)PD7
- net LCD_RS: now also IC1.PC5(A13/OC.3B), U1.PC5(A13/OC.3B); no longer U1.(INT6/AIN0)PE6
- net M0_A: now also IC1.PA3(AD3), U1.PA3(AD3); no longer U1.(ADC11/PCINT4)PB4
- net M0_B: now also IC1.PA6(AD6), U1.PA6(AD6); no longer U1.(PCINT7/OC0A/OC1C/#RTS)PB7
- net M1_A: now also IC1.PA4(AD4), U1.PA4(AD4); no longer U1.(PCINT5/OC1A/#OC4B/ADC12)PB5
- net M1_B: now also IC1.PA7(AD7), U1.PA7(AD7); no longer U1.(T1/#OC4D/ADC9)PD6
- net M2_A: now also IC1.PA5(AD5), U1.PA5(AD5); no longer U1.(PCINT6/OC1B/OC4B/ADC13)PB6
- net M2_B: now also IC1.PB0(SS/PCINT0), U1.PB0(SS/PCINT0); no longer U1.(ICP3/CLK0/OC4A)PC7
- net RD+: now also IC1.D+
- net RD-: now also IC1.D-
- net SHT: now also IC1.PD5(XCK1), U1.PD5(XCK1); no longer U1.(ADC1)PF1
- net UCAP: now also C22.2, IC1.UCAP; no longer C6.1
- net VIN: now also R25.2
- net VUSB: now also IC1.VBUS
Other:
- moved on the sheet: C1, C14, C2, C21, C3, C4, C5, C6, JMP, R11, X1

Commit message: finished routing. needs optimizing for SDB
Parts:
- removed C14: .1uF, parkers_parts:CAP_NONPOL0402
- removed H3: MOUNT-HOLE3.0, holes:MOUNT-HOLE3.0
- removed R27: 10K, parkers_parts:RESISTOR0402
- removed S1, S2: SKHHAJA010, SparkFun-Electromechanical:SWITCH-MOMENTARY-2PTH
- JMP: value (none) -> P1X02PH; device parkers_parts:RESISTOR0402 -> parkers_parts:P1X02PH
Connections:
- removed net PE3: IC1.PE3(IUID), U1.PE3(IUID)
- removed net PE7: IC1.PE7(INT7/AIN1/UVCON), U1.PE7(INT7/AIN1/UVCON)
- new net PD5: IC1.PD5(XCK1), U1.PD5(XCK1)
- new net PD6: IC1.PD6(T1), U1.PD6(T1)
- net +5V: now also JMP.2; no longer C14.1, JMP.1, R27.1
- net COM1: now also IC1.PD7(T0), U1.PD7(T0); no longer IC1.PD0(OC.0B/SCL/INT0), U1.PD0(OC.0B/SCL/INT0)
- net COM3: now also IC1.PD0(OC.0B/SCL/INT0), U1.PD0(OC.0B/SCL/INT0); no longer IC1.PD7(T0), U1.PD7(T0)
- net FOC: now also IC1.PE7(INT7/AIN1/UVCON), U1.PE7(INT7/AIN1/UVCON); no longer IC1.PD6(T1), U1.PD6(T1)
- net GND: no longer C14.2, S1.2, S2.2
- net PE2: no longer R27.2, S2.1
- net RST: no longer S1.1
- net SHT: now also IC1.PE3(IUID), U1.PE3(IUID); no longer IC1.PD5(XCK1), U1.PD5(XCK1)
- net VUSB: now also JMP.1; no longer JMP.2

Commit message: finished SDB REV2
Parts:
- removed R25: 36K, parkers_parts:RESISTOR0402
- removed R26: 20K, parkers_parts:RESISTOR0402
- added C14: .1uF, parkers_parts:CAP_NONPOL0402
- added D2: PMEG6010EP, parkers_parts:DIODESOD-128
- added U10: IP4234CZ6, parkers_parts:IP4234CZ6SOT-457
- C10, C11, C8: value .1uF -> .1uF 35V
- D1: value PMEG3030EP -> PMEG6010EP
- J4: value RJHS-538X -> RJHSE-5381
- MOT0, MOT1, MOT2: value (none) -> KLDX-0202-B-LT
- PWR: value (none) -> KLDX-0202-A-LT
- R4: value 22 -> 4K
- R5: value 22 -> 20K
- renumbered IC1 to U11
Connections:
- net 12VB: now also D2.CATHODE
- net BATT_V: now also C14.1, R4.2, R5.1; no longer R25.1, R26.2
- net COM1: now also CG4.1
- net COM2: now also CG7.1
- net COM3: now also CG1.2
- net D+: now also U10.I/O1A; no longer CG1.2, R5.1
- net D-: now also U10.I/O2B; no longer CG2.2, R4.1
- net GND: now also C14.2, CG1.1, CG2.1, CG4.2, CG7.2, D2.ANODE, R4.1; no longer CG4.1, R26.1
- net IO_2: now also CG2.2; no longer CG3.2
- net IO_3: now also CG3.2; no longer CG4.2
- net RD+: now also U10.I/O1B; no longer R5.2
- net RD-: now also U10.I/O2A; no longer R4.2
- net UGND: now also U10.GND; no longer CG1.1, CG2.1, CG7.1
- net VIN: now also R5.2; no longer R25.2
- net VUSB: now also U10.VB; no longer CG7.2
Other:
- moved on the sheet: CG1, CG2, CG3, CG4, CG7, R4, R5

Commit message: finished REV2 of SDB
Parts:
- added AUX: (no value), pinhead:PINHD-2X4
- added CG8, CG9: CG0402MLC-05LG, parkers_parts:RESISTOR0402
- added J6: SJ1-2503A, parkers_parts:TRS_STEREO_JACKSJ1-2503A
- LCD1: value LCD-16X2 -> LCD-16X2NOHOLES; device SparkFun:LCD-16X2 -> SparkFun-Displays:LCD-16X2NOHOLES
- U$1: REVNUM 1 -> 2
Connections:
- removed net PE4: U1.PE4(INT4/TOSC1), U11.PE4(INT4/TOSC1)
- removed net PE5: U1.PE5(INT5/TOSC2), U11.PE5(INT5/TOSC2)
- removed net PE6: U1.PE6(INT6/AIN0), U11.PE6(INT6/AIN0)
- new net PB5: U1.PB5(PCINT5/OC.1A), U11.PB5(PCINT5/OC.1A)
- new net PB6: U1.PB6(PCINT6/OC.1B), U11.PB6(PCINT6/OC.1B)
- new net PD7: U1.PD7(T0), U11.PD7(T0)
- net +5V: now also AUX.1
- net COM1: now also U1.PB4(PCINT4/OC.2A), U11.PB4(PCINT4/OC.2A); no longer U1.PD7(T0), U11.PD7(T0)
- net FOC: now also U1.PB7(PCINT7/OC.0A/OC.1C), U11.PB7(PCINT7/OC.0A/OC.1C); no longer U1.PE7(INT7/AIN1/UVCON), U11.PE7(INT7/AIN1/UVCON)
- net GND: now also AUX.2, CG8.1, CG9.1, J6.S
- net IO_0: now also CG8.2, J6.T, U1.PE4(INT4/TOSC1), U11.PE4(INT4/TOSC1); no longer U1.PB4(PCINT4/OC.2A), U11.PB4(PCINT4/OC.2A)
- net IO_1: now also CG9.2, J6.R, U1.PE5(INT5/TOSC2), U11.PE5(INT5/TOSC2); no longer U1.PB5(PCINT5/OC.1A), U11.PB5(PCINT5/OC.1A)
- net IO_2: now also U1.PE6(INT6/AIN0), U11.PE6(INT6/AIN0); no longer U1.PB6(PCINT6/OC.1B), U11.PB6(PCINT6/OC.1B)
- net IO_3: now also U1.PE7(INT7/AIN1/UVCON), U11.PE7(INT7/AIN1/UVCON); no longer U1.PB7(PCINT7/OC.0A/OC.1C), U11.PB7(PCINT7/OC.0A/OC.1C)
- net PF2: now also AUX.3
- net PF3: now also AUX.4
- net PF4: now also AUX.5
- net PF5: now also AUX.6
- net PF6: now also AUX.7
- net PF7: now also AUX.8

Commit message: REV 3 of SDB in works. Fixed the pull up on the BTNS, changes RS485 chip to one with ESD built in.
Parts:
- removed JMP: P1X02PH, parkers_parts:P1X02PH
- removed U8: TPD2E007DCK, parkers_parts:TPD2E007DCK
- added C24: 100uF, PP_Passives:CAPACITOR_POLARIZED6.3MM_SMD
- added R25: 10K, parkers_parts:RESISTOR0402
- R13: value 68 -> 100
- R16: value 43 -> 100
- U$1: REVNUM 2 -> 3
- U6: value SN75176BDR -> ISL8483
Connections:
- removed net VUSB: J1.VBUS, JMP.1, U1.VBUS, U10.VB, U11.VBUS
- net +5V: now also J1.VBUS, R15.1, R25.1, U1.VBUS, U10.VB, U11.VBUS; no longer JMP.2, R10.2
- net A: no longer U8.IO2
- net B: no longer U8.IO1
- net BTNS: now also R25.2
- net GND: now also C24.NEG; no longer U8.GND
- net OK_SHT: now also R10.2; no longer R15.1
- net VIN: now also C24.POS

Commit message: REV 7 of the USB Board done. Moving to production on it.
SDB Rev 3 almost done. OTG USB added. Motor controllers switched to BTM7755 to reduce the Resistance on of the drivers.
Parts:
- removed C22: 1uF, parkers_parts:CAP_NONPOL0402
- removed C23: .1uF, parkers_parts:CAP_NONPOL0402
- removed C24: 100uF, PP_Passives:CAPACITOR_POLARIZED6.3MM_SMD
- added CG10: CG0402MLC-05LG, parkers_parts:RESISTOR0402
- added R26, R29: 4.7K, parkers_parts:RESISTOR0402
- added R27, R28, R30, R31, R32, R33, R34: 10K, parkers_parts:RESISTOR0402
- C12: value .1uF -> 100uF; device parkers_parts:CAP_NONPOL0402 -> PP_Passives:CAPACITOR_POLARIZED6.3MM_SMD
- C15: value .1uF -> 1uF
- C9: value .1uF -> .1uF 35V
- MOT0, MOT1, MOT2, PWR: device parkers_parts:DC_JACKPTH -> PP_Connectors:DC_JACKPTH_TIGHT
- R1, R2, R7, R8: value 10K -> 4.7K
- U3: value TB6559FG -> BTM7755; device parkers_parts:TB6559FG -> PP_PowerIC:BTM7755PG-DSO-36-29
- U5, U7: value TB6559FG -> (none); device parkers_parts:TB6559FG -> PP_PowerIC:BTM7755PG-DSO-36-29
Connections:
- removed net N$15: C15.1, U5.VREG
- removed net N$19: C13.1, U7.VREG
- removed net N$40: C12.1, U3.VREG
- removed net PB5: U1.PB5(PCINT5/OC.1A), U11.PB5(PCINT5/OC.1A)
- new net N$1: R7.1, U5.IN2
- new net N$10: R1.1, U3.IN2
- new net N$2: R8.1, U5.IN1
- new net N$3: R26.1, U5.INH
- new net N$4: R3.1, U7.IN2
- new net N$6: R6.1, U7.IN1
- new net N$7: R32.1, U7.INH
- new net N$8: R29.1, U3.INH
- new net N$9: R2.1, U3.IN1
- new net PE3: CG10.2, U1.PE3(IUID), U11.PE3(IUID)
- net +5V: no longer U3.SB, U3.VREF, U5.SB, U5.VREF, U7.SB, U7.VREF
- net AGND: now also C13.2; no longer C23.2
- net AREF: now also C13.1; no longer C23.1
- net GND: now also C10.1, C11.1, C12.NEG, C9.1, CG10.1, R27.2, R28.2, R30.2, R31.2, R33.2, R34.2; no longer C10.2, C11.2, C12.2, C13.2, C15.2, C24.NEG, C9.2, R1.1, R2.1, R3.1, R6.1, R7.1, R8.1, U3.RSA, U5.RSA, U7.RSA
- net M0_A: now also R7.2; no longer R8.2, U5.IN1
- net M0_B: now also R8.2, U1.PA4(AD4), U11.PA4(AD4); no longer R7.2, U1.PA6(AD6), U11.PA6(AD6), U5.IN2
- net M0_O1: now also R27.1
- net M0_O2: now also R28.1
- net M0_P: now also R26.2; no longer U5.PWM
- net M1_A: now also R3.2, U1.PA5(AD5), U11.PA5(AD5); no longer R6.2, U1.PA4(AD4), U11.PA4(AD4), U7.IN1
- net M1_B: now also R6.2, U1.PA6(AD6), U11.PA6(AD6); no longer R3.2, U1.PA7(AD7), U11.PA7(AD7), U7.IN2
- net M1_O1: now also R34.1
- net M1_O2: now also R33.1
- net M1_P: now also R32.2; no longer U7.PWM
- net M2_A: now also R1.2, U1.PA7(AD7), U11.PA7(AD7); no longer R2.2, U1.PA5(AD5), U11.PA5(AD5), U3.IN1
- net M2_B: now also R2.2; no longer R1.2, U3.IN2
- net M2_O1: now also R31.1
- net M2_O2: now also R30.1
- net M2_P: now also R29.2; no longer U3.PWM
- net SHT: now also U1.PB5(PCINT5/OC.1A), U11.PB5(PCINT5/OC.1A); no longer U1.PE3(IUID), U11.PE3(IUID)
- net UCAP: now also C15.2; no longer C22.2
- net UGND: now also C15.1; no longer C22.1
- net VIN: now also C10.2, C11.2, C12.POS, C9.2, U3.VS, U5.VS, U7.VS; no longer C10.1, C11.1, C24.POS, C9.1, U3.VCC, U5.VCC, U7.VCC
Other:
- moved on the sheet: C10, C11, C13, C15, C9, MOT0, MOT1, MOT2, R1, R2, R3, R6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

Commit message: added 0805 package to pp_passives for resistors. changed resistors on the motor output lines from 0402 to 0805 for better heat dissipation.
Parts:
- R27, R28, R30, R31, R33, R34: device parkers_parts:RESISTOR0402 -> PP_Passives:RESISTOR0805
Changed lines of the file:
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@@
 <grid distance="0.1" unitdist="inch" unit="inch" style="lines" multiple="1" display="no" altdistance="0.01" altunitdist="inch" altunit="inch"/>
 <layers>
-<layer number="1" name="Top" color="4" fill="1" visible="yes" active="no"/>
-<layer number="2" name="Route2" color="1" fill="3" visible="yes" active="no"/>
-<layer number="3" name="Route3" color="4" fill="3" visible="yes" active="no"/>
-<layer number="4" name="Route4" color="1" fill="4" visible="yes" active="no"/>
-<layer number="5" name="Route5" color="4" fill="4" visible="yes" active="no"/>
-<layer number="6" name="Route6" color="1" fill="8" visible="yes" active="no"/>
-<layer number="7" name="Route7" color="4" fill="8" visible="yes" active="no"/>
-<layer number="8" name="Route8" color="1" fill="2" visible="yes" active="no"/>
-<layer number="9" name="Route9" color="4" fill="2" visible="yes" active="no"/>
-<layer number="10" name="Route10" color="1" fill="7" visible="yes" active="no"/>
-<layer number="11" name="Route11" color="4" fill="7" visible="yes" active="no"/>
-<layer number="12" name="Route12" color="1" fill="5" visible="yes" active="no"/>
-<layer number="13" name="Route13" color="4" fill="5" visible="yes" active="no"/>
-<layer number="14" name="Route14" color="1" fill="6" visible="yes" active="no"/>
-<layer number="15" name="Route15" color="4" fill="6" visible="yes" active="no"/>
-<layer number="16" name="Bottom" color="1" fill="1" visible="yes" active="no"/>
-<layer number="17" name="Pads" color="2" fill="1" visible="yes" active="no"/>
-<layer number="18" name="Vias" color="10" fill="1" visible="yes" active="no"/>
-<layer number="19" name="Unrouted" color="6" fill="1" visible="yes" active="no"/>
-<layer number="20" name="Dimension" color="15" fill="1" visible="yes" active="no"/>
-<layer number="21" name="tPlace" color="7" fill="1" visible="yes" active="no"/>
-<layer number="22" name="bPlace" color="7" fill="1" visible="yes" active="no"/>
-<layer number="23" name="tOrigins" color="15" fill="1" visible="yes" active="no"/>
-<layer number="24" name="bOrigins" color="15" fill="1" visible="yes" active="no"/>
-<layer number="25" name="tNames" color="7" fill="1" visible="yes" active="no"/>
-<layer number="26" name="bNames" color="7" fill="1" visible="yes" active="no"/>
-<layer number="27" name="tValues" color="7" fill="1" visible="yes" active="no"/>
-<layer number="28" name="bValues" color="7" fill="1" visible="yes" active="no"/>
+<layer number="1" name="Top" color="4" fill="1" visible="no" active="no"/>
+<layer number="2" name="Route2" color="1" fill="3" visible="no" active="no"/>
+<layer number="3" name="Route3" color="4" fill="3" visible="no" active="no"/>
+<layer number="4" name="Route4" color="1" fill="4" visible="no" active="no"/>
+<layer number="5" name="Route5" color="4" fill="4" visible="no" active="no"/>
+<layer number="6" name="Route6" color="1" fill="8" visible="no" active="no"/>
+<layer number="7" name="Route7" color="4" fill="8" visible="no" active="no"/>
+<layer number="8" name="Route8" color="1" fill="2" visible="no" active="no"/>
+<layer number="9" name="Route9" color="4" fill="2" visible="no" active="no"/>
+<layer number="10" name="Route10" color="1" fill="7" visible="no" active="no"/>
+<layer number="11" name="Route11" color="4" fill="7" visible="no" active="no"/>
+<layer number="12" name="Route12" color="1" fill="5" visible="no" active="no"/>
+<layer number="13" name="Route13" color="4" fill="5" visible="no" active="no"/>
+<layer number="14" name="Route14" color="1" fill="6" visible="no" active="no"/>
+<layer number="15" name="Route15" color="4" fill="6" visible="no" active="no"/>
+<layer number="16" name="Bottom" color="1" fill="1" visible="no" active="no"/>
+<layer number="17" name="Pads" color="2" fill="1" visible="no" active="no"/>
+<layer number="18" name="Vias" color="10" fill="1" visible="no" active="no"/>
+<layer number="19" name="Unrouted" color="6" fill="1" visible="no" active="no"/>
+<layer number="20" name="Dimension" color="15" fill="1" visible="no" active="no"/>
+<layer number="21" name="tPlace" color="7" fill="1" visible="no" active="no"/>
+<layer number="22" name="bPlace" color="7" fill="1" visible="no" active="no"/>
+<layer number="23" name="tOrigins" color="15" fill="1" visible="no" active="no"/>
+<layer number="24" name="bOrigins" color="15" fill="1" visible="no" active="no"/>
+<layer number="25" name="tNames" color="7" fill="1" visible="no" active="no"/>
+<layer number="26" name="bNames" color="7" fill="1" visible="no" active="no"/>
+<layer number="27" name="tValues" color="7" fill="1" visible="no" active="no"/>
+<layer number="28" name="bValues" color="7" fill="1" visible="no" active="no"/>
 <layer number="29" name="tStop" color="2" fill="3" visible="no" active="no"/>
 <layer number="30" name="bStop" color="5" fill="6" visible="no" active="no"/>
@@
 <layer number="35" name="tGlue" color="7" fill="4" visible="no" active="no"/>
 <layer number="36" name="bGlue" color="7" fill="5" visible="no" active="no"/>
-<layer number="37" name="tTest" color="7" fill="1" visible="yes" active="no"/>
-<layer number="38" name="bTest" color="7" fill="1" visible="yes" active="no"/>
+<layer number="37" name="tTest" color="7" fill="1" visible="no" active="no"/>
+<layer number="38" name="bTest" color="7" fill="1" visible="no" active="no"/>
 <layer number="39" name="tKeepout" color="4" fill="11" visible="no" active="no"/>
 <layer number="40" name="bKeepout" color="1" fill="11" visible="no" active="no"/>
@@
 <layer number="44" name="Drills" color="7" fill="1" visible="no" active="no"/>
 <layer number="45" name="Holes" color="7" fill="1" visible="no" active="no"/>
-<layer number="46" name="Milling" color="3" fill="1" visible="yes" active="no"/>
-<layer number="47" name="Measures" color="7" fill="1" visible="yes" active="no"/>
-<layer number="48" name="Document" color="7" fill="1" visible="yes" active="no"/>
-<layer number="49" name="Reference" color="13" fill="1" visible="yes" active="no"/>
-<layer number="50" name="dxf" color="12" fill="1" visible="yes" active="no"/>
-<layer number="51" name="tDocu" color="7" fill="1" visible="yes" active="no"/>
-<layer number="52" name="bDocu" color="7" fill="1" visible="yes" active="no"/>
-<layer number="53" name="tGND_GNDA" color="7" fill="1" visible="yes" active="no"/>
-<layer number="54" name="bGND_GNDA" color="7" fill="1" visible="yes" active="no"/>
-<layer number="56" name="wert" color="7" fill="1" visible="yes" active="no"/>
+<layer number="46" name="Milling" color="3" fill="1" visible="no" active="no"/>
+<layer number="47" name="Measures" color="7" fill="1" visible="no" active="no"/>
+<layer number="48" name="Document" color="7" fill="1" visible="no" active="no"/>
+<layer number="49" name="Reference" color="13" fill="1" visible="no" active="no"/>
+<layer number="50" name="dxf" color="12" fill="1" visible="no" active="no"/>
+<layer number="51" name="tDocu" color="7" fill="1" visible="no" active="no"/>
+<layer number="52" name="bDocu" color="7" fill="1" visible="no" active="no"/>
+<layer number="53" name="tGND_GNDA" color="7" fill="1" visible="no" active="no"/>
+<layer number="54" name="bGND_GNDA" color="7" fill="1" visible="no" active="no"/>
+<layer number="56" name="wert" color="7" fill="1" visible="no" active="no"/>
 <layer number="91" name="Nets" color="2" fill="1" visible="yes" active="yes"/>
 <layer number="92" name="Busses" color="1" fill="1" visible="yes" active="yes"/>
@@
 <part name="U7" library="PP_PowerIC" deviceset="BTM7755" device="PG-DSO-36-29"/>
 <part name="R26" library="parkers_parts" deviceset="RESISTOR" device="0402" value="4.7K"/>
-<part name="R27" library="parkers_parts" deviceset="RESISTOR" device="0402" value="10K"/>
-<part name="R28" library="parkers_parts" deviceset="RESISTOR" device="0402" value="10K"/>
+<part name="R27" library="PP_Passives" deviceset="RESISTOR" device="0805" value="10K"/>
+<part name="R28" library="PP_Passives" deviceset="RESISTOR" device="0805" value="10K"/>
 <part name="R29" library="parkers_parts" deviceset="RESISTOR" device="0402" value="4.7K"/>
-<part name="R30" library="parkers_parts" deviceset="RESISTOR" device="0402" value="10K"/>
-<part name="R31" library="parkers_parts" deviceset="RESISTOR" device="0402" value="10K"/>
+<part name="R30" library="PP_Passives" deviceset="RESISTOR" device="0805" value="10K"/>
+<part name="R31" library="PP_Passives" deviceset="RESISTOR" device="0805" value="10K"/>
 <part name="R32" library="parkers_parts" deviceset="RESISTOR" device="0402" value="10K"/>
-<part name="R33" library="parkers_parts" deviceset="RESISTOR" device="0402" value="10K"/>
-<part name="R34" library="parkers_parts" deviceset="RESISTOR" device="0402" value="10K"/>
+<part name="R33" library="PP_Passives" deviceset="RESISTOR" device="0805" value="10K"/>
+<part name="R34" library="PP_Passives" deviceset="RESISTOR" device="0805" value="10K"/>
 <part name="CG10" library="parkers_parts" deviceset="RESISTOR" device="0402" value="CG0402MLC-05LG"/>
 </parts>
