File: Super_Dolly_Board.sch (EAGLE design)
At the start: 101 parts, among them J1 10118193-0001LF, J3 SJ1-2503A, J4 RJHSE-5381, J5 SJ1-2503A, J6 SJ1-2503A, P1 TC33X-2, SW1 SKQUDBE010, U1 AT90USB646-MU, U10 IP4234CZ6, U11 AT90USB646-AU, U2 MMDT3904, U3 BTM7755, U4 TS2937CW50, U6 ISL8483, U9 TS2937CW50, X1 3.2X2.5MMCRYSTAL

Commit message: Tagged SDB REV_3
Connections:
- net N$1 renamed M0_A1
- net N$2 renamed M0_B1
- net N$3 renamed M0_P1
Changed lines of the file:
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@@
 </segment>
 </net>
-<net name="N$3" class="0">
+<net name="M0_P1" class="0">
 <segment>
 <pinref part="R26" gate="G$1" pin="1"/>
@@
 </segment>
 </net>
-<net name="N$1" class="0">
+<net name="M0_A1" class="0">
 <segment>
 <pinref part="R7" gate="G$1" pin="1"/>
@@
 </segment>
 </net>
-<net name="N$2" class="0">
+<net name="M0_B1" class="0">
 <segment>
 <pinref part="R8" gate="G$1" pin="1"/>
