File: Super_Dolly_Board.sch (EAGLE design)
At the start: 106 parts, among them J1 10118193-0001LF, J3 SJ1-2503A, J4 RJHSE-5381, J5 SJ1-2503A, J6 SJ1-2503A, J7 HFW6R-2STE1LF, P1 TC33X-2, U1 AT90USB646-MU, U10 IP4234CZ6, U11 AT90USB646-AU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

Commit message: Fixed some small isues with the SDM REV4 and tagged it as REV5. Added the spreadsheet BOM.
Parts:
- added U15: MC78M05CDTG, PP_PowerIC:FIXED_VOLTAGE_REGDPAK-3
- CG1, CG10, CG2, CG3, CG4, CG5, CG6, CG7, CG8, CG9: value TPD1E10B06DPYR -> CG0402MLC-05LG
- U$1: REVNUM 4 -> 5
- renumbered C23 to C20
Connections:
- new net 12VB_D: D2.CATHODE, U15.IN
- net +5V: now also U15.OUT
- net GND: now also U15.GND
- net VIN: no longer D2.CATHODE
