File: Tribble.sch (EAGLE design)
At the start: 106 parts, among them J1 10118193-0001LF, J2 68602-406HLF, J3 SJ1-2503A, J4 RJHSE-5381, J5 SJ1-2503A, J6 SJ1-2503A, J7 HFW6R-2STE1LF, P1 TC33X-2, U1 AT90USB646-MU, U10 IP4234CZ6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

Commit message: Fixing EMC problems with Tribble. Moved lots of traces. Added Ferrite beads to COM1, COM2, Com3. Added proper support for USB OTG
Parts:
- added C23: .1uF, parkers_parts:CAP_NONPOL0402
- added C24: 10uF, SparkFun:CAP_POL1206
- added D3: PMEG3010BER,115, PP_Passives:DIODESOD-123
- added F2: 1206L025YR, PP_Passives:PTC_FUSE1206
- added FB1, FB2, FB3: LI0402C470R-10, parkers_parts:RESISTOR0402
- added R38, R39: 22, parkers_parts:RESISTOR0402
- added R40: 100K, parkers_parts:RESISTOR0402
- added R41: 10K, parkers_parts:RESISTOR0402
- added U15: BC847BMTF, PP_DiscreteSemi:BJT_NPN_SINGLESOT-23
- added U16: FDV304P, PP_DiscreteSemi:MOSFET_P-CHANNEL_SINGLESOT-23
- J1: device SparkFun-Connectors:USB-PTH-MICROB -> PP_Connectors:USB10118193-0001LF
- U$1: REVNUM 6 -> 7
- U10: device parkers_parts:IP4234CZ6SOT-457 -> PP_Passives:IP4234CZ6SOT-457
Connections:
- removed net PE0: U1.PE0(/WR), U11.PE0(/WR)
- new net COM1_FB: CG4.1, FB1.1, J4.3
- new net COM2_FB: CG7.1, FB2.1, J4.4
- new net COM3_FB: CG1.2, FB3.1, J4.8
- new net FDV_GATE: R41.2, U15.COLLECTOR, U16.GATE
- new net N$11: R38.1, U10.I/O2B
- new net N$13: R39.1, U10.I/O2A
- new net N$14: D3.CATHODE, F2.P$1
- new net PE7: R40.2, U1.PE7(INT7/AIN1/UVCON), U11.PE7(INT7/AIN1/UVCON)
- new net PE7_GATE: R40.1, U15.BASE
- new net V_USB: C23.2, D3.ANODE, J1.5V, U1.VBUS, U10.VB, U11.VBUS, U16.DRAIN
- net +5V: now also C24.+, F2.P$2, R41.1, U16.SOURCE; no longer J1.VBUS, U1.VBUS, U10.VB, U11.VBUS
- net COM1: now also FB1.2; no longer CG4.1, J4.3
- net COM2: now also FB2.2; no longer CG7.1, J4.4
- net COM3: now also FB3.2; no longer CG1.2, J4.8
- net D-: now also U10.I/O1B; no longer U10.I/O2B
- net GND: now also C24.-, U15.EMITTER
- net IO_3: now also U1.PE0(/WR), U11.PE0(/WR); no longer U1.PE7(INT7/AIN1/UVCON), U11.PE7(INT7/AIN1/UVCON)
- net PE3: now also J1.ID
- net RD+: now also R39.2; no longer U10.I/O1B
- net RD-: now also R38.2; no longer U10.I/O2A
- net UGND: now also C23.1, CG10.1
Other:
- moved on the sheet: D1, PWR, R22, R37, U10, U12

Commit message: updated the BOM info for Tribble Rev 7
Parts:
- CG1, CG10, CG2, CG3, CG4, CG5, CG6, CG7, CG8, CG9: value CG0402MLC-05LG -> B72590D50H260
- D3: value PMEG3010BER,115 -> PMEG6010EP,115; device PP_Passives:DIODESOD-123 -> PP_Passives:DIODESOD-128
- U1: value AT90USB646-MU -> AT90USB1287-MU
- U11: value AT90USB646-AU -> AT90USB1287-AU
- U12: value FDS6681Z -> FDS6679AZ
- X1: value CX3225SB16000D0FLJZZ -> TSX-3225 16.0000MF10U-B0

Commit message: Fixed the issues for Tribble that popped up during EMC testing
Parts:
- added C25: 100uF, PP_Passives:CAPACITOR_POLARIZED6.3MM_SMD
- added C26: 100uF, PP_Passives:CAPACITOR_POLARIZED5MM_SMD
- FB1, FB2, FB3: value LI0402C470R-10 -> HZ0402B102R-10
- U$1: REVNUM 7 -> 8
Connections:
- net +5V: now also C26.POS
- net GND: now also C25.NEG, C26.NEG
- net VIN: now also C25.POS
Other:
- note added: "CG = Chip Gaurd / ESD Protection"

Commit message: tagged loads of PCBs and made sure BOMs where up to date
Parts:
- added D4: P6SMB30CAT3G, PP_Passives:DIODEDO-214AA
- added TVS1, TVS2, TVS3, TVS4: ESD11B5.0ST5G, PP_Passives:TVS_DIODEDSN-2
Connections:
- net +5V: now also TVS1.P$2, TVS2.P$2, TVS3.P$2, TVS4.P$2
- net GND: now also D4.ANODE, TVS1.P$1, TVS2.P$1, TVS3.P$1, TVS4.P$1
- net VIN_J: now also D4.CATHODE
Other:
- moved on the sheet: D1, F1, F2, R37, U12

Commit message: Revert to REV 7 of Tribble
Did not need the board fixes in REV 8 of the pcb.
Parts:
- removed C25: 100uF, PP_Passives:CAPACITOR_POLARIZED6.3MM_SMD
- removed C26: 100uF, PP_Passives:CAPACITOR_POLARIZED5MM_SMD
- removed D4: P6SMB30CAT3G, PP_Passives:DIODEDO-214AA
- removed TVS1, TVS2, TVS3, TVS4: ESD11B5.0ST5G, PP_Passives:TVS_DIODEDSN-2
- FB1, FB2, FB3: value HZ0402B102R-10 -> LI0402C470R-10
- U$1: REVNUM 8 -> 7
Connections:
- net +5V: no longer C26.POS, TVS1.P$2, TVS2.P$2, TVS3.P$2, TVS4.P$2
- net GND: no longer C25.NEG, C26.NEG, D4.ANODE, TVS1.P$1, TVS2.P$1, TVS3.P$1, TVS4.P$1
- net VIN: no longer C25.POS
- net VIN_J: no longer D4.CATHODE
Other:
- note removed: "CG = Chip Gaurd / ESD Protection"
- moved on the sheet: D1, F1, F2, R37, U12
